File: interface.kicad_sch (KiCad schematic)
At the start: 1 part, among them J2 Conn_01x16

Commit message: Add files via upload
Parts:
- added C12: 100n, Capacitor_SMD:C_0603_1608Metric, symbol Device:C_Small
- added C14: 1n, Capacitor_SMD:C_0603_1608Metric, symbol Device:C_Small
- added C9: 1u, Capacitor_SMD:C_0603_1608Metric, symbol Device:C_Small
- added FB2: Bead, Inductor_SMD:L_0603_1608Metric, symbol Device:FerriteBead_Small
- added R2 (x3): 10k, Resistor_SMD:R_0603_1608Metric, symbol Device:R_Small
- renumbered J2 to J3
Connections:
- net nRST: now reaches J3.1 (Pin_1)
- net nRST: now also R2.1
- net PA_ENA: now reaches J3.12 (Pin_12)
- net FWD_SENSE: now reaches J3.13 (Pin_13)
- net REF_SENSE: now reaches J3.14 (Pin_14)
- net GND: now reaches J3.15 (Pin_15)
- net GND: now also J3.16 (Pin_16), C12.2, C14.2, C9.2, R2.2
- net SPI_MISO: now reaches J3.2 (Pin_2)
- net SPI_MOSI: now reaches J3.3 (Pin_3)
- net SPI_SCK: now reaches J3.4 (Pin_4)
- net TX_nCS: now reaches J3.5 (Pin_5)
- net TX_nCS: now also R2.1
- net RX_nCS: now reaches J3.6 (Pin_6)
- net RX_nCS: now also R2.1
- net MCU_TX: now reaches J3.7 (Pin_7)
- net MCU_RX: now reaches J3.8 (Pin_8)
- new net 3V3_IN: C9.1, FB2.1
- new net INTERFACE_3V3: C12.1, C14.1, FB2.2, R2.2, R2.2
- no-connect marks 0 -> 3
Other:
- note added: "Decoupling"
- note added: "External connector"
- moved on the sheet: J3

Commit message: Add files via upload
Connections:
- net PA_ENA renamed PA_EN
Changed lines of the file:
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@@
     (effects (font (size 1.27 1.27)) (justify left))
   )
-  (hierarchical_label "PA_ENA" (shape output) (at 146.05 151.13 0) (fields_autoplaced)
+  (hierarchical_label "PA_EN" (shape output) (at 146.05 151.13 0) (fields_autoplaced)
     (effects (font (size 1.27 1.27)) (justify left))
   )

Commit message: Add files via upload
Parts:
- renumbered J3 to J4
Changed lines of the file:
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@@
         )
         (path "/4c42207c-9e6b-42da-ad38-da126b892014/3ea647a3-6e2c-4a7a-bdb8-a6b94119ef02"
-          (reference "R35") (unit 1)
+          (reference "R38") (unit 1)
         )
       )
@@
   (symbol (lib_id "Connector_Generic:Conn_01x16") (at 109.22 140.97 0) (mirror y) (unit 1)
     (in_bom yes) (on_board yes) (dnp no) (fields_autoplaced)
-    (property "Reference" "J3" (at 109.22 117.7757 0)
+    (property "Reference" "J4" (at 109.22 117.7757 0)
       (effects (font (size 1.27 1.27)))
     )
@@
       (project "m17-rru-rf"
         (path "/4c42207c-9e6b-42da-ad38-da126b892014/3ea647a3-6e2c-4a7a-bdb8-a6b94119ef02"
-          (reference "J3") (unit 1)
+          (reference "J4") (unit 1)
         )
       )
@@
         )
         (path "/4c42207c-9e6b-42da-ad38-da126b892014/3ea647a3-6e2c-4a7a-bdb8-a6b94119ef02"
-          (reference "R37") (unit 1)
+          (reference "R40") (unit 1)
         )
       )
@@
         )
         (path "/4c42207c-9e6b-42da-ad38-da126b892014/3ea647a3-6e2c-4a7a-bdb8-a6b94119ef02"
-          (reference "#PWR085") (unit 1)
+          (reference "#PWR0104") (unit 1)
         )
       )
@@
         )
         (path "/4c42207c-9e6b-42da-ad38-da126b892014/3ea647a3-6e2c-4a7a-bdb8-a6b94119ef02"
-          (reference "#PWR087") (unit 1)
+          (reference "#PWR0106") (unit 1)
         )
       )
@@
         )
         (path "/4c42207c-9e6b-42da-ad38-da126b892014/3ea647a3-6e2c-4a7a-bdb8-a6b94119ef02"
-          (reference "R36") (unit 1)
+          (reference "R39") (unit 1)
         )
       )
@@
         )
         (path "/4c42207c-9e6b-42da-ad38-da126b892014/3ea647a3-6e2c-4a7a-bdb8-a6b94119ef02"
-          (reference "#PWR086") (unit 1)
+          (reference "#PWR0105") (unit 1)
         )
       )
@@
         )
         (path "/4c42207c-9e6b-42da-ad38-da126b892014/3ea647a3-6e2c-4a7a-bdb8-a6b94119ef02"
-          (reference "C69") (unit 1)
+          (reference "C83") (unit 1)
         )
       )
@@
         )
         (path "/4c42207c-9e6b-42da-ad38-da126b892014/3ea647a3-6e2c-4a7a-bdb8-a6b94119ef02"
-          (reference "C67") (unit 1)
+          (reference "C81") (unit 1)
         )
       )
@@
         )
         (path "/4c42207c-9e6b-42da-ad38-da126b892014/3ea647a3-6e2c-4a7a-bdb8-a6b94119ef02"
-          (reference "FB5") (unit 1)
+          (reference "FB7") (unit 1)
         )
       )
@@
         )
         (path "/4c42207c-9e6b-42da-ad38-da126b892014/3ea647a3-6e2c-4a7a-bdb8-a6b94119ef02"
-          (reference "C68") (unit 1)
+          (reference "C82") (unit 1)
         )
       )
@@
         )
         (path "/4c42207c-9e6b-42da-ad38-da126b892014/3ea647a3-6e2c-4a7a-bdb8-a6b94119ef02"
-          (reference "#PWR089") (unit 1)
+          (reference "#PWR0108") (unit 1)
         )
       )
@@
         )
         (path "/4c42207c-9e6b-42da-ad38-da126b892014/3ea647a3-6e2c-4a7a-bdb8-a6b94119ef02"
-          (reference "#PWR088") (unit 1)
-        )
-      )
+          (reference "#PWR0107") (unit 1)
+        )
+      )

Commit message: Add files via upload
Parts:
- renumbered J4 to J5
Other:
- note added: "Add ESD protection"
- note added: "All devices held in reset state while nRST remains unconnected"
Changed lines of the file:
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@@
     (effects (font (size 3.81 3.81)) (justify left bottom))
+  )
+  (text "All devices held in reset state\nwhile nRST remains unconnected"
+    (at 78.74 109.22 0)
+    (effects (font (size 1.27 1.27)) (justify left bottom))
+  )
+  (text "Add ESD protection" (at 125.73 162.56 0)
+    (effects (font (size 1.27 1.27)) (justify left bottom))
   )
   (label "INTERFACE_3V3" (at 146.05 104.14 0) (fields_autoplaced)
@@
         )
         (path "/4c42207c-9e6b-42da-ad38-da126b892014/3ea647a3-6e2c-4a7a-bdb8-a6b94119ef02"
-          (reference "R38") (unit 1)
+          (reference "R41") (unit 1)
         )
       )
@@
   (symbol (lib_id "Connector_Generic:Conn_01x16") (at 109.22 140.97 0) (mirror y) (unit 1)
     (in_bom yes) (on_board yes) (dnp no) (fields_autoplaced)
-    (property "Reference" "J4" (at 109.22 117.7757 0)
+    (property "Reference" "J5" (at 109.22 117.7757 0)
       (effects (font (size 1.27 1.27)))
     )
@@
       (project "m17-rru-rf"
         (path "/4c42207c-9e6b-42da-ad38-da126b892014/3ea647a3-6e2c-4a7a-bdb8-a6b94119ef02"
-          (reference "J4") (unit 1)
+          (reference "J5") (unit 1)
         )
       )
@@
         )
         (path "/4c42207c-9e6b-42da-ad38-da126b892014/3ea647a3-6e2c-4a7a-bdb8-a6b94119ef02"
-          (reference "R40") (unit 1)
+          (reference "R43") (unit 1)
         )
       )
@@
         )
         (path "/4c42207c-9e6b-42da-ad38-da126b892014/3ea647a3-6e2c-4a7a-bdb8-a6b94119ef02"
-          (reference "#PWR0104") (unit 1)
+          (reference "#PWR0105") (unit 1)
         )
       )
@@
         )
         (path "/4c42207c-9e6b-42da-ad38-da126b892014/3ea647a3-6e2c-4a7a-bdb8-a6b94119ef02"
-          (reference "#PWR0106") (unit 1)
+          (reference "#PWR0107") (unit 1)
         )
       )
@@
         )
         (path "/4c42207c-9e6b-42da-ad38-da126b892014/3ea647a3-6e2c-4a7a-bdb8-a6b94119ef02"
-          (reference "R39") (unit 1)
+          (reference "R42") (unit 1)
         )
       )
@@
         )
         (path "/4c42207c-9e6b-42da-ad38-da126b892014/3ea647a3-6e2c-4a7a-bdb8-a6b94119ef02"
-          (reference "#PWR0105") (unit 1)
+          (reference "#PWR0106") (unit 1)
         )
       )
@@
         )
         (path "/4c42207c-9e6b-42da-ad38-da126b892014/3ea647a3-6e2c-4a7a-bdb8-a6b94119ef02"
+          (reference "#PWR0109") (unit 1)
+        )
+      )
+    )
+  )
+  (symbol (lib_id "power:GND") (at 283.21 139.7 0) (unit 1)
+    (in_bom yes) (on_board yes) (dnp no) (fields_autoplaced)
+    (property "Reference" "#PWR027" (at 283.21 146.05 0)
+      (effects (font (size 1.27 1.27)) hide)
+    )
+    (property "Value" "GND" (at 283.21 143.8331 0)
+      (effects (font (size 1.27 1.27)))
+    )
+    (property "Footprint" "" (at 283.21 139.7 0)
+      (effects (font (size 1.27 1.27)) hide)
+    )
+    (property "Datasheet" "" (at 283.21 139.7 0)
+      (effects (font (size 1.27 1.27)) hide)
+    )
+    (pin "1")
+    (instances
+      (project "m17-rru-rf"
+        (path "/4c42207c-9e6b-42da-ad38-da126b892014/ccc39fee-262d-4ac9-a9a6-59e024db6eed"
+          (reference "#PWR027") (unit 1)
+        )
+        (path "/4c42207c-9e6b-42da-ad38-da126b892014/3ea647a3-6e2c-4a7a-bdb8-a6b94119ef02"
           (reference "#PWR0108") (unit 1)
         )
       )
-    )
-  )
-  (symbol (lib_id "power:GND") (at 283.21 139.7 0) (unit 1)
-    (in_bom yes) (on_board yes) (dnp no) (fields_autoplaced)
-    (property "Reference" "#PWR027" (at 283.21 146.05 0)
-      (effects (font (size 1.27 1.27)) hide)
-    )
-    (property "Value" "GND" (at 283.21 143.8331 0)
-      (effects (font (size 1.27 1.27)))
-    )
-    (property "Footprint" "" (at 283.21 139.7 0)
-      (effects (font (size 1.27 1.27)) hide)
-    )
-    (property "Datasheet" "" (at 283.21 139.7 0)
-      (effects (font (size 1.27 1.27)) hide)
-    )
-    (pin "1")
-    (instances
-      (project "m17-rru-rf"
-        (path "/4c42207c-9e6b-42da-ad38-da126b892014/ccc39fee-262d-4ac9-a9a6-59e024db6eed"
-          (reference "#PWR027") (unit 1)
-        )
-        (path "/4c42207c-9e6b-42da-ad38-da126b892014/3ea647a3-6e2c-4a7a-bdb8-a6b94119ef02"
-          (reference "#PWR0107") (unit 1)
-        )
-      )

Commit message: partial PN update
Parts:
- C12: PN (none) -> C0603C104M5RAC7411
- C14: PN (none) -> C0603C102J5GAC7411
- C9: PN (none) -> CL10B105KB8NQNC
Changed lines of the file:
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@@
+      (effects (font (size 1.27 1.27)) hide)
+    )
+    (property "PN" "C0603C102J5GAC7411" (at 292.1 134.62 0)
       (effects (font (size 1.27 1.27)) hide)
     )
@@
         )
         (path "/4c42207c-9e6b-42da-ad38-da126b892014/3ea647a3-6e2c-4a7a-bdb8-a6b94119ef02"
-          (reference "C83") (unit 1)
+          (reference "C84") (unit 1)
         )
       )
@@
       (effects (font (size 1.27 1.27)) hide)
     )
+    (property "PN" "CL10B105KB8NQNC" (at 271.78 134.62 0)
+      (effects (font (size 1.27 1.27)) hide)
+    )
     (pin "1")
     (pin "2")
@@
         )
         (path "/4c42207c-9e6b-42da-ad38-da126b892014/3ea647a3-6e2c-4a7a-bdb8-a6b94119ef02"
-          (reference "C81") (unit 1)
+          (reference "C82") (unit 1)
         )
       )
@@
       (effects (font (size 1.27 1.27)) hide)
     )
+    (property "PN" "C0603C104M5RAC7411" (at 283.21 134.62 0)
+      (effects (font (size 1.27 1.27)) hide)
+    )
     (pin "1")
     (pin "2")
@@
         )
         (path "/4c42207c-9e6b-42da-ad38-da126b892014/3ea647a3-6e2c-4a7a-bdb8-a6b94119ef02"
-          (reference "C82") (unit 1)
+          (reference "C83") (unit 1)
         )
       )
