File: mcu.kicad_sch (KiCad schematic)
At the start: 1 part, among them U12 STM32F405RGTx

Commit message: Add files via upload
Parts:
- renumbered U12 to U13
Changed lines of the file:
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@@
     (comment 1 "Wojciech Kaczmarski, SP5WWP")
+  )
+  (hierarchical_label "MCU_TX" (shape output) (at 101.6 129.54 0) (fields_autoplaced)
+    (effects (font (size 1.27 1.27)) (justify left))
+  )
+  (hierarchical_label "MCU_RX" (shape input) (at 101.6 133.35 0) (fields_autoplaced)
+    (effects (font (size 1.27 1.27)) (justify left))
   )
   (symbol (lib_id "MCU_ST_STM32F4:STM32F405RGTx") (at 144.78 99.06 0) (unit 1)
     (in_bom yes) (on_board yes) (dnp no) (fields_autoplaced)
-    (property "Reference" "U12" (at 149.5141 143.9601 0)
+    (property "Reference" "U13" (at 149.5141 143.9601 0)
       (effects (font (size 1.27 1.27)) (justify left))
     )
@@
       (project "m17-rru-rf"
         (path "/4c42207c-9e6b-42da-ad38-da126b892014/270fa747-1697-46c9-b996-5c9733c883e2"
-          (reference "U12") (unit 1)
+          (reference "U13") (unit 1)
         )
       )

Commit message: Add files via upload
Changed lines of the file:
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@@
     (comment 1 "Wojciech Kaczmarski, SP5WWP")
+  )
+  (hierarchical_label "RF_PWR_SP" (shape output) (at 205.74 134.62 0) (fields_autoplaced)
+    (effects (font (size 1.27 1.27)) (justify left))
   )
   (hierarchical_label "MCU_TX" (shape output) (at 101.6 129.54 0) (fields_autoplaced)

Commit message: Add files via upload
Parts:
- added C12 (x2): 100n, Capacitor_SMD:C_0603_1608Metric, symbol Device:C_Small
- added C14 (x2): 1n, Capacitor_SMD:C_0603_1608Metric, symbol Device:C_Small
- added C9 (x2): 1u, Capacitor_SMD:C_0603_1608Metric, symbol Device:C_Small
- added C9 (x2): 2u2, Capacitor_SMD:C_0603_1608Metric, symbol Device:C_Small
- added FB2 (x2): Bead, Inductor_SMD:L_0603_1608Metric, symbol Device:FerriteBead_Small
- added J5: Conn_01x05, symbol Connector_Generic:Conn_01x05
Connections:
- net MCU_3V3: now reaches U13.1 (VBAT)
- net MCU_3V3: now also U13.19 (VDD), U13.32 (VDD), U13.48 (VDD), U13.64 (VDD), C12.1, C14.1, FB2.2, J5.5 (Pin_5)
- net GND: now reaches U13.12 (VSSA)
- net GND: now also U13.18 (VSS), U13.60 (BOOT0), U13.63 (VSS), C12.2, C12.2, C14.2, C14.2, C9.2, C9.2, C9.2, C9.2, J5.1 (Pin_1)
- net MCU_VDDA_3V3: now reaches U13.13 (VDDA)
- net MCU_VDDA_3V3: now also C12.1, C14.1, FB2.2
- net at U13.31 (VCAP_1): now also C9.1
- net at U13.47 (VCAP_2): now also C9.1
- net nRST: now reaches U13.7 (NRST)
- net nRST: now also J5.2 (Pin_2)
- new net 3V3_IN: C9.1, C9.1, FB2.1, FB2.1
- new net SWDCLK: J5.4 (Pin_4)
- new net SWDIO: J5.3 (Pin_3)
Other:
- note added: "Decoupling"
- note added: "SWD"

Commit message: Add files via upload
Parts:
- added C12 (x4): 100n, Capacitor_SMD:C_0603_1608Metric, symbol Device:C_Small
- added C9 (x2): 10p, Capacitor_SMD:C_0603_1608Metric, symbol Device:C_Small
- added R2 (x3): 100R, Resistor_SMD:R_0603_1608Metric, symbol Device:R_Small
- added Y1: 12MHz, Crystal:Crystal_SMD_3225-4Pin_3.2x2.5mm, symbol Device:Crystal_GND24_Small
- C14: value 1n -> 10n
- J3: renamed from J5; footprint (none) -> Connector_PinHeader_2.54mm:PinHeader_1x05_P2.54mm_Vertical_SMD_Pin1Left
Connections:
- net GND: now also C12.2, C12.2, C12.2, C12.2, C9.2, C9.2, Y1.2, Y1.4
- net MCU_3V3: now also C12.1, C12.1, C12.1, C12.1
- net MCU_RX: now also U13.43 (PA10)
- net MCU_TX: now also U13.42 (PA9)
- net RF_PWR_SP: now also U13.20 (PA4)
- net SWDCLK: now also U13.49 (PA14)
- net SWDIO: now also U13.46 (PA13)
- net FWD_SENSE: now reaches U13.14 (PA0)
- net REF_SENSE: now reaches U13.15 (PA1)
- net AIN2: now reaches U13.16 (PA2)
- net AIN3: now reaches U13.17 (PA3)
- net AOUT1: now reaches U13.21 (PA5)
- net OSC1: now reaches U13.5 (PH0)
- net OSC1: now also C9.1, Y1.1
- net at U13.55 (PB3): now also R2.1
- net at U13.56 (PB4): now also R2.1
- net at U13.57 (PB5): now also R2.1
- net RX_nCS: now reaches U13.58 (PB6)
- net TX_nCS: now reaches U13.59 (PB7)
- net OSC2: now reaches U13.6 (PH1)
- net OSC2: now also C9.1, Y1.3
- net PA_EN: now reaches U13.61 (PB8)
- new net SPI_MISO: R2.2
- new net SPI_MOSI: R2.2
- new net SPI_SCK: R2.2
- no-connect marks 0 -> 3
Other:
- note added: "MCU"
- note added: "Place close to the MCU"
- moved on the sheet: C12, C14, C9, FB2, J3, U13

Commit message: Add files via upload
Parts:
- added J3: Conn_01x05, Connector_PinHeader_2.54mm:PinHeader_1x05_P2.54mm_Vertical_SMD_Pin1Left, symbol Connector_Generic:Conn_01x05
- renumbered J3 to J4
Connections:
- net GND: now also J3.5 (Pin_5)
- net TP1: now reaches U13.27 (PB1)
- net TP1: now also J3.1 (Pin_1)
- net TP2: now reaches U13.28 (PB2)
- net TP2: now also J3.2 (Pin_2)
- net DBG_TX: now reaches U13.29 (PB10)
- net DBG_TX: now also J3.3 (Pin_3)
- net DBG_RX: now reaches U13.30 (PB11)
- net DBG_RX: now also J3.4 (Pin_4)
- no-connect marks 3 -> 29

Commit message: partial PN update
Parts:
- C12: PN (none) -> C0603C104M5RAC7411
- C14: PN (none) -> C0603C103K5RAC7081
- C9: PN (none) -> CL10B105KB8NQNC
- C9: PN (none) -> GRM188R61H225ME11J
