File: rf_pa.kicad_sch (KiCad schematic)
At the start: 52 parts, among them Q1 BSS138, Q2 BSS138, Q3 NP100P04PDG, U1 LT1013DIDR, U2 LM317_SOT-223, U3 TL431, U4 RA60H3847H1

Commit message: PN update
Parts:
- FB1: PN (none) -> BLM18KG601SH1D
- TP1, TP10, TP2, TP3, TP4, TP5, TP6, TP7, TP8, TP9: value ~ -> TP; PN (none) -> -
- U1: PN (none) -> LT1013DIDR
- U4: PN (none) -> -
Changed lines of the file:
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@@
       (effects (font (size 1.27 1.27)) (justify left))
     )
-    (property "Value" "~" (at 146.05 75.8246 0)
+    (property "Value" "TP" (at 146.05 75.8246 0)
       (effects (font (size 1.27 1.27)) (justify left))
     )
@@
     )
     (property "Datasheet" "~" (at 147.32 76.2 0)
+      (effects (font (size 1.27 1.27)) hide)
+    )
+    (property "PN" "-" (at 142.24 76.2 0)
       (effects (font (size 1.27 1.27)) hide)
     )
@@
       (effects (font (size 1.27 1.27)) hide)
     )
+    (property "PN" "-" (at 284.48 95.25 0)
+      (effects (font (size 1.27 1.27)) hide)
+    )
     (pin "1")
     (pin "2")
@@
       (effects (font (size 1.27 1.27)) (justify left))
     )
-    (property "Value" "~" (at 163.83 183.7746 0)
+    (property "Value" "TP" (at 163.83 183.7746 0)
       (effects (font (size 1.27 1.27)) (justify left))
     )
@@
       (effects (font (size 1.27 1.27)) hide)
     )
+    (property "PN" "-" (at 160.02 184.15 0)
+      (effects (font (size 1.27 1.27)) hide)
+    )
     (pin "1")
     (instances
@@
       (effects (font (size 1.27 1.27)) (justify left))
     )
-    (property "Value" "~" (at 82.55 111.3846 0)
+    (property "Value" "TP" (at 82.55 111.3846 0)
       (effects (font (size 1.27 1.27)) (justify left))
     )
@@
       (effects (font (size 1.27 1.27)) hide)
     )
+    (property "PN" "-" (at 78.74 111.76 0)
+      (effects (font (size 1.27 1.27)) hide)
+    )
     (pin "1")
     (instances
@@
       (effects (font (size 1.27 1.27)) (justify left))
     )
-    (property "Value" "~" (at 152.4 110.1146 0)
+    (property "Value" "TP" (at 152.4 110.1146 0)
       (effects (font (size 1.27 1.27)) (justify left))
     )
@@
     )
     (property "Datasheet" "~" (at 151.13 110.49 0)
+      (effects (font (size 1.27 1.27)) hide)
+    )
+    (property "PN" "-" (at 156.21 110.49 0)
       (effects (font (size 1.27 1.27)) hide)
     )
@@
       (effects (font (size 1.27 1.27)) hide)
     )
-    (property "PN" "" (at 146.05 187.96 90)
+    (property "PN" "BLM18KG601SH1D" (at 146.05 187.96 90)
       (effects (font (size 1.27 1.27)) hide)
     )
@@
     (property "Manufacturer_Part_Number" "LT1013DIDR" (at 129.54 891.44 0)
       (effects (font (size 1.27 1.27)) (justify left top) hide)
+    )
+    (property "PN" "LT1013DIDR" (at 100.33 96.52 0)
+      (effects (font (size 1.27 1.27)) hide)
     )
     (pin "1")
@@
       (effects (font (size 1.27 1.27)) (justify left))
     )
-    (property "Value" "~" (at 190.5 113.9246 0)
+    (property "Value" "TP" (at 190.5 113.9246 0)
       (effects (font (size 1.27 1.27)) (justify left))
     )
@@
       (effects (font (size 1.27 1.27)) hide)
     )
+    (property "PN" "-" (at 186.69 114.3 0)
+      (effects (font (size 1.27 1.27)) hide)
+    )
     (pin "1")
     (instances
@@
       (effects (font (size 1.27 1.27)) (justify left))
     )
-    (property "Value" "~" (at 142.24 113.9246 0)
+    (property "Value" "TP" (at 142.24 113.9246 0)
       (effects (font (size 1.27 1.27)) (justify left))
     )
@@
       (effects (font (size 1.27 1.27)) hide)
     )
+    (property "PN" "-" (at 138.43 114.3 0)
+      (effects (font (size 1.27 1.27)) hide)
+    )
     (pin "1")
     (instances
@@
       (effects (font (size 1.27 1.27)) (justify left))
     )
-    (property "Value" "~" (at 269.24 181.2346 0)
+    (property "Value" "TP" (at 269.24 181.2346 0)
       (effects (font (size 1.27 1.27)) (justify left))
     )
@@
       (effects (font (size 1.27 1.27)) hide)
     )
+    (property "PN" "-" (at 265.43 181.61 0)
+      (effects (font (size 1.27 1.27)) hide)
+    )
     (pin "1")
     (instances
@@
       (effects (font (size 1.27 1.27)))
     )
-    (property "Value" "~" (at 271.4046 171.45 0)
+    (property "Value" "TP" (at 271.4046 171.45 0)
       (effects (font (size 1.27 1.27)) (justify left))
     )
@@
       (effects (font (size 1.27 1.27)) hide)
     )
+    (property "PN" "-" (at 271.78 175.26 0)
+      (effects (font (size 1.27 1.27)) hide)
+    )
     (pin "1")
     (instances
@@
       (effects (font (size 1.27 1.27)) (justify left))
     )
-    (property "Value" "~" (at 78.3646 81.28 0)
+    (property "Value" "TP" (at 78.3646 81.28 0)
       (effects (font (size 1.27 1.27)) (justify left))
     )
@@
       (effects (font (size 1.27 1.27)) hide)
     )
+    (property "PN" "-" (at 78.74 85.09 0)
+      (effects (font (size 1.27 1.27)) hide)
+    )
     (pin "1")
     (instances
@@
       (effects (font (size 1.27 1.27)) (justify left))
     )
-    (property "Value" "~" (at 269.24 206.6346 0)
+    (property "Value" "TP" (at 269.24 206.6346 0)
       (effects (font (size 1.27 1.27)) (justify left))
     )
@@
       (effects (font (size 1.27 1.27)) hide)
     )
+    (property "PN" "-" (at 265.43 207.01 0)
+      (effects (font (size 1.27 1.27)) hide)
+    )
