File: m17-rru-rf.kicad_pcb (KiCad board)
At the start: 4 copper layers, 240 x 150 mm, 68 parts, among them J1 Conn_Coaxial, J2 Conn_01x16, Q1 BSS138, Q2 NP100P04PDG, U1 LM317_SOT-223, U10 AD8318ACPZ-REEL7, U11 AD8318ACPZ-REEL7, U12 STM32F405RGTx, U2 LT1013DIDR, U3 TL431, U4 RA60H3847H1, U5 CC1200, U9 CC1200

Commit message: Add files via upload
Parts:
- added C18: 1n, Capacitor_SMD:C_0603_1608Metric, F.Cu at (132.6, 115.8)
- added C19: 47n, Capacitor_SMD:C_0603_1608Metric, F.Cu at (132.6, 118.3)
- added C20: 1n5, Capacitor_SMD:C_0603_1608Metric, F.Cu at (132.6, 120.8)
- added C21: 47n, Capacitor_SMD:C_0603_1608Metric, F.Cu at (132.6, 123.3)
- added C22: 47n, Capacitor_SMD:C_0603_1608Metric, F.Cu at (132.6, 125.8)
- added C23: 47n, Capacitor_SMD:C_0603_1608Metric, F.Cu at (132.6, 128.3)
- added C24: 47n, Capacitor_SMD:C_0603_1608Metric, F.Cu at (132.6, 130.8)
- added C25: 47n, Capacitor_SMD:C_0603_1608Metric, F.Cu at (132.6, 133.3)
- added C26: 47n, Capacitor_SMD:C_0603_1608Metric, F.Cu at (136.6, 115.8)
- added C27: 47n, Capacitor_SMD:C_0603_1608Metric, F.Cu at (136.6, 118.3)
- added C28: 100n, Capacitor_SMD:C_0603_1608Metric, F.Cu at (136.6, 120.8)
- added C29: 47n, Capacitor_SMD:C_0603_1608Metric, F.Cu at (136.6, 123.3)
- added C30: 47n, Capacitor_SMD:C_0603_1608Metric, F.Cu at (136.6, 125.8)
- added C31: 47n, Capacitor_SMD:C_0603_1608Metric, F.Cu at (136.6, 128.3)
- added C32: 39p, Capacitor_SMD:C_0603_1608Metric, F.Cu at (136.6, 130.8)
- added C33: 56p, Capacitor_SMD:C_0603_1608Metric, F.Cu at (136.6, 133.3)
- added C34: 2p2, Capacitor_SMD:C_0603_1608Metric, F.Cu at (140.6, 115.8)
- added C35: 10n, Capacitor_SMD:C_0603_1608Metric, F.Cu at (140.6, 118.3)
- added C36: 5p1, Capacitor_SMD:C_0603_1608Metric, F.Cu at (140.6, 120.8)
- added C37: 100p, Capacitor_SMD:C_0603_1608Metric, F.Cu at (140.6, 123.3)
- added C38: 6n2, Capacitor_SMD:C_0603_1608Metric, F.Cu at (140.6, 125.8)
- added C39: 1u, Capacitor_SMD:C_0603_1608Metric, F.Cu at (155.0, 125.7)
- added C40: 100n, Capacitor_SMD:C_0603_1608Metric, F.Cu at (155.0, 128.2)
- added C41: 1n, Capacitor_SMD:C_0603_1608Metric, F.Cu at (155.0, 130.7)
- added C42: 100n, Capacitor_SMD:C_0603_1608Metric, F.Cu at (155.0, 133.2)
- added C43: 1n, Capacitor_SMD:C_0603_1608Metric, F.Cu at (155.0, 135.8)
- added C44: 1n, Capacitor_SMD:C_0603_1608Metric, F.Cu at (159.1, 125.7)
- added C45: 100n, Capacitor_SMD:C_0603_1608Metric, F.Cu at (159.1, 128.2)
- added C46: 1n, Capacitor_SMD:C_0603_1608Metric, F.Cu at (159.1, 130.7)
- added C47: 1n, Capacitor_SMD:C_0603_1608Metric, F.Cu at (159.1, 133.2)
- added C48: 1u, Capacitor_SMD:C_0603_1608Metric, F.Cu at (126.5, 115.8)
- added C49: 100n, Capacitor_SMD:C_0603_1608Metric, F.Cu at (126.5, 118.3)
- added C50: 1n, Capacitor_SMD:C_0603_1608Metric, F.Cu at (126.5, 120.8)
- added FB3: Bead, Inductor_SMD:L_0603_1608Metric, F.Cu at (159.1, 135.8)
- added FB4: Bead, Inductor_SMD:L_0603_1608Metric, F.Cu at (126.5, 123.3)
- added J3: Conn_01x16, Connector_PinHeader_2.54mm:PinHeader_2x08_P2.54mm_Vertical_SMD, F.Cu at (64.8, 135.9)
- added L1: 10u, Inductor_SMD:L_Vishay_IHLP-2525, F.Cu at (158.0, 118.5)
- added L2: 56n, Inductor_SMD:L_0603_1608Metric, F.Cu at (140.6, 128.3)
- added L3: 15n, Inductor_SMD:L_0603_1608Metric, F.Cu at (140.6, 130.8)
- added L4: 43n, Inductor_SMD:L_0603_1608Metric, F.Cu at (140.6, 133.3)
- added L5: 22n, Inductor_SMD:L_0603_1608Metric, F.Cu at (153.7, 102.9)
- added R23: 100R, Resistor_SMD:R_0603_1608Metric, F.Cu at (144.6, 118.3)
- added R24: 56k, Resistor_SMD:R_0603_1608Metric, F.Cu at (144.6, 120.8)
- added R25: 18R, Resistor_SMD:R_0603_1608Metric, F.Cu at (144.6, 123.3)
- added R26: 52R3, Resistor_SMD:R_0603_1608Metric, F.Cu at (163.1, 125.7)
- added R27: 499R, Resistor_SMD:R_0603_1608Metric, F.Cu at (163.1, 128.2)
- added R28: 52R3, Resistor_SMD:R_0603_1608Metric, F.Cu at (163.1, 130.7)
- added R29: 499R, Resistor_SMD:R_0603_1608Metric, F.Cu at (163.1, 133.2)
- added R30: ~, Parts:HALF_FLANGE_DUMMY_LOAD, F.Cu at (293.6, 88.3)
- added R31: 10k, Resistor_SMD:R_0603_1608Metric, F.Cu at (126.5, 125.8)
- added R32: 10k, Resistor_SMD:R_0603_1608Metric, F.Cu at (126.5, 128.3)
- added R33: 10k, Resistor_SMD:R_0603_1608Metric, F.Cu at (126.5, 130.8)
- added TP7: ~, TestPoint:TestPoint_Pad_D1.5mm, F.Cu at (164.7, 116.3)
- added TP8: ~, TestPoint:TestPoint_Pad_D1.5mm, F.Cu at (164.7, 119.8)
- added U14: ~, Parts:CIRC_H08, F.Cu at (264.2, 88.9)
- added X1: 40MHz, Oscillator:Oscillator_SMD_SeikoEpson_SG210-4Pin_2.5x2.0mm, F.Cu at (148.8, 116.4)
- C10: value 100n -> 22u/6.3V
- C11: value 1n -> 100n
- C13: value 1n -> 100u/50V; footprint Capacitor_SMD:C_0603_1608Metric -> Capacitor_SMD:CP_Elec_8x10.5
- C14: value 1n -> 22u/6.3V
- C15: value 100n -> 47n
- C16, C17: value 1n -> 47n
- C9: value 1u -> 100u/50V; footprint Capacitor_SMD:C_0603_1608Metric -> Capacitor_SMD:CP_Elec_8x10.5
- J1: value Conn_Coaxial -> Conn_01x01_Pin; footprint Connector_Coaxial:SMA_Samtec_SMA-J-P-X-ST-EM1_EdgeMount -> TestPoint:TestPoint_Pad_D3.0mm
- J2: value Conn_01x16 -> Conn_Coaxial; footprint Connector_PinHeader_2.54mm:PinHeader_2x08_P2.54mm_Vertical_SMD -> Connector_Coaxial:SMA_Samtec_SMA-J-P-X-ST-EM1_EdgeMount
- R18: value 52R3 -> 100k
- R19: value 499R -> 24k
- R20: value 52R3 -> 75k
- R21: value 499R -> 100R
- R22: value ~ -> 100R; footprint Parts:HALF_FLANGE_DUMMY_LOAD -> Resistor_SMD:R_0603_1608Metric
- U10: value AD8318ACPZ-REEL7 -> CC1200; footprint Mine:QFN65P400X400X100-17N -> Package_DFN_QFN:QFN-32-1EP_5x5mm_P0.5mm_EP3.45x3.45mm
- U12: value STM32F405RGTx -> AD8318ACPZ-REEL7; footprint Package_QFP:LQFP-64_10x10mm_P0.5mm -> Mine:QFN65P400X400X100-17N
- U13: value ~ -> STM32F405RGTx; footprint Parts:CIRC_H08 -> Package_QFP:LQFP-64_10x10mm_P0.5mm
- U5: value CC1200 -> ~; footprint Package_DFN_QFN:QFN-32-1EP_5x5mm_P0.5mm_EP3.45x3.45mm -> Package_TO_SOT_SMD:SOT-23-6
- U6: value ~ -> CC1200; footprint Parts:GAT-30_LAND -> Package_DFN_QFN:QFN-32-1EP_5x5mm_P0.5mm_EP3.45x3.45mm
- U7: footprint Parts:SYBD-30_LAND -> Parts:GAT-30_LAND
- U8: footprint Parts:GAT-30_LAND -> Parts:SYBD-30_LAND
- U9: value CC1200 -> ~; footprint Package_DFN_QFN:QFN-32-1EP_5x5mm_P0.5mm_EP3.45x3.45mm -> Parts:GAT-30_LAND
- moved R21 129.8 mm to (285.8, 163.8), turned to 90 degrees
- moved U8 2.62 mm to (125.7, 196.8)
Connections:
- C10 pad 1: Net-(U10-CLPF) -> GND
- C10 pad 2: GND -> /Power supply/13.8V_OUT
- C11 pad 1: GND -> /Power supply/13.8V_OUT
- C11 pad 2: Net-(U10-INLO) -> GND
- C12 pad 1: /RF detectors/RF_DET_3V3 -> Net-(U5-BST)
- C12 pad 2: GND -> Net-(U5-SW)
- C13 pad 1: /RF coupler/FWD_SENSE -> /Power supply/13.8V_OUT
- C13 pad 2: Net-(U10-INHI) -> GND
- C14 pad 1: /RF detectors/RF_DET_3V3 -> GND
- C14 pad 2: GND -> /Exciter/3.3V_IN
- C15 pad 1: Net-(U11-CLPF) -> /Exciter/EXCITER_3V3
- C16 pad 1: GND -> /Exciter/EXCITER_3V3
- C16 pad 2: Net-(U11-INLO) -> GND
- C17 pad 1: /RF coupler/REF_SENSE -> /Exciter/EXCITER_3V3
- C17 pad 2: Net-(U11-INHI) -> GND
- C9 pad 1: /Exciter/3.3V_IN -> /RF PA/RF_PA_VDD
- FB2 pad 1: /Exciter/3.3V_IN -> /Exciter/EXCITER_3V3
- FB2 pad 2: /RF detectors/RF_DET_3V3 -> /Exciter/3.3V_IN
- J1 pad 1: Net-(J1-In) -> /Power supply/13.8V_OUT
- J2 pad 1: unconnected-(J2-Pin_1-Pad1) -> Net-(J2-In)
- J2 pad 2: unconnected-(J2-Pin_2-Pad2) -> GND
- R18 pad 1: GND -> /Power supply/13.8V_OUT
- R18 pad 2: /RF coupler/FWD_SENSE -> Net-(U5-EN)
- R19 pad 1: Net-(U10-TADJ) -> Net-(U5-FB)
- R20 pad 1: GND -> Net-(U5-FB)
- R20 pad 2: /RF coupler/REF_SENSE -> /Exciter/3.3V_IN
- R21 pad 1: Net-(U11-TADJ) -> Net-(U6-SCLK)
- R21 pad 2: GND -> /Exciter/SPI_SCK
- R22 pad 1: Net-(R22-In) -> Net-(U6-SI)
- U10 pad 1: GND -> unconnected-(U10-VDD_GUARD-Pad1)
- U10 pad 10: Net-(U10-TADJ) -> unconnected-(U10-GPIO0-Pad10)
- U10 pad 11: GND -> unconnected-(U10-~{CS}-Pad11)
- U10 pad 12: GND -> unconnected-(U10-DVDD-Pad12)
- U10 pad 14: Net-(U10-INHI) -> unconnected-(U10-RBIAS-Pad14)
- U10 pad 15: Net-(U10-INLO) -> unconnected-(U10-AVDD_RF-Pad15)
- U10 pad 16: /RF detectors/RF_DET_3V3 -> (no net)
- U10 pad 17: GND -> unconnected-(U10-PA-Pad17)
- U10 pad 2: GND -> unconnected-(U10-~{RESET}-Pad2)
- U10 pad 3: /RF detectors/RF_DET_3V3 -> unconnected-(U10-GPIO3-Pad3)
- U10 pad 4: /RF detectors/RF_DET_3V3 -> unconnected-(U10-GPIO2-Pad4)
- U10 pad 5: Net-(U10-CLPF) -> unconnected-(U10-DVDD-Pad5)
- U10 pad 6: /RF PA/FWD_SENSE_IN -> unconnected-(U10-DCPL-Pad6)
- U10 pad 7: /RF PA/FWD_SENSE_IN -> unconnected-(U10-SI-Pad7)
- U10 pad 8: GND -> unconnected-(U10-SCLK-Pad8)
- U10 pad 9: /RF detectors/RF_DET_3V3 -> unconnected-(U10-SO(GPIO1)-Pad9)
- U11 pad 6: /RF detectors/RF_REF_DET -> /RF PA/FWD_SENSE_IN
- U11 pad 7: /RF detectors/RF_REF_DET -> /RF PA/FWD_SENSE_IN
- U12 pad 1: unconnected-(U12-VBAT-Pad1) -> GND
- U12 pad 10: unconnected-(U12-PC2-Pad10) -> Net-(U12-TADJ)
- U12 pad 11: unconnected-(U12-PC3-Pad11) -> GND
- U12 pad 12: unconnected-(U12-VSSA-Pad12) -> GND
- U12 pad 14: unconnected-(U12-PA0-Pad14) -> Net-(U12-INHI)
- U12 pad 15: unconnected-(U12-PA1-Pad15) -> Net-(U12-INLO)
- U12 pad 16: unconnected-(U12-PA2-Pad16) -> /RF detectors/RF_DET_3V3
- U12 pad 17: unconnected-(U12-PA3-Pad17) -> GND
- U12 pad 2: unconnected-(U12-PC13-Pad2) -> GND
- U12 pad 3: unconnected-(U12-PC14-Pad3) -> /RF detectors/RF_DET_3V3
- U12 pad 4: unconnected-(U12-PC15-Pad4) -> /RF detectors/RF_DET_3V3
- U12 pad 5: unconnected-(U12-PH0-Pad5) -> Net-(U12-CLPF)
- U12 pad 6: unconnected-(U12-PH1-Pad6) -> /RF detectors/RF_REF_DET
- U12 pad 7: unconnected-(U12-NRST-Pad7) -> /RF detectors/RF_REF_DET
- U12 pad 8: unconnected-(U12-PC0-Pad8) -> GND
- U12 pad 9: unconnected-(U12-PC1-Pad9) -> /RF detectors/RF_DET_3V3
- U13 pad 1: /Circulator/RF_IN -> unconnected-(U13-VBAT-Pad1)
- U13 pad 2: /Circulator/RF_OUT -> unconnected-(U13-PC13-Pad2)
- U13 pad 3: Net-(R22-In) -> unconnected-(U13-PC14-Pad3)
- U5 pad 1: unconnected-(U5-VDD_GUARD-Pad1) -> Net-(U5-BST)
- U5 pad 2: unconnected-(U5-~{RESET}-Pad2) -> GND
- U5 pad 3: unconnected-(U5-GPIO3-Pad3) -> Net-(U5-FB)
- U5 pad 4: unconnected-(U5-GPIO2-Pad4) -> Net-(U5-EN)
- U5 pad 5: unconnected-(U5-DVDD-Pad5) -> /Power supply/13.8V_OUT
- U5 pad 6: unconnected-(U5-DCPL-Pad6) -> Net-(U5-SW)
- U6 pad 1: Net-(U6-In) -> /Exciter/EXCITER_3V3
- U6 pad 2: GND -> /Exciter/nRST
- U6 pad 3: /RF coupler/REF_SENSE -> unconnected-(U6-GPIO3-Pad3)
- U6 pad 4: GND -> unconnected-(U6-GPIO2-Pad4)
- U7 pad 1: Net-(J1-In) -> Net-(U7-In)
- U7 pad 2: /Circulator/RF_OUT -> GND
- U7 pad 3: Net-(U7-Rev) -> /RF coupler/REF_SENSE
- U7 pad 4: Net-(U6-In) -> GND
- U8 pad 1: Net-(U7-Rev) -> Net-(J2-In)
- U8 pad 2: GND -> /Circulator/RF_OUT
- U8 pad 3: /RF coupler/FWD_SENSE -> Net-(U8-Rev)
- U8 pad 4: GND -> Net-(U7-In)
- U9 pad 1: unconnected-(U9-VDD_GUARD-Pad1) -> Net-(U8-Rev)
- U9 pad 2: unconnected-(U9-~{RESET}-Pad2) -> GND
- U9 pad 3: unconnected-(U9-GPIO3-Pad3) -> /RF coupler/FWD_SENSE
- U9 pad 4: unconnected-(U9-GPIO2-Pad4) -> GND

Commit message: Add files via upload
Parts:
- added C51: 47n, Capacitor_SMD:C_0603_1608Metric, F.Cu at (216.0, 174.1)
- added C52: 5p1, Capacitor_SMD:C_0603_1608Metric, F.Cu at (216.0, 176.6)
- added C53: 47n, Capacitor_SMD:C_0603_1608Metric, F.Cu at (216.0, 179.1)
- added C54: 47n, Capacitor_SMD:C_0603_1608Metric, F.Cu at (216.0, 181.6)
- added C55: 5p1, Capacitor_SMD:C_0603_1608Metric, F.Cu at (220.0, 174.1)
- added C56: 6p2, Capacitor_SMD:C_0603_1608Metric, F.Cu at (220.0, 176.6)
- added C57: 47n, Capacitor_SMD:C_0603_1608Metric, F.Cu at (220.0, 179.1)
- added C58: 1u, Capacitor_SMD:C_0603_1608Metric, F.Cu at (210.0, 154.5)
- added C59: 100n, Capacitor_SMD:C_0603_1608Metric, F.Cu at (210.0, 157.0)
- added C60: 1n, Capacitor_SMD:C_0603_1608Metric, F.Cu at (210.0, 159.5)
- added C61: 100n, Capacitor_SMD:C_0603_1608Metric, F.Cu at (210.0, 162.0)
- added C62: 1n, Capacitor_SMD:C_0603_1608Metric, F.Cu at (210.0, 164.6)
- added C63: 1n, Capacitor_SMD:C_0603_1608Metric, F.Cu at (210.0, 167.1)
- added C64: 100n, Capacitor_SMD:C_0603_1608Metric, F.Cu at (210.0, 169.6)
- added C65: 1n, Capacitor_SMD:C_0603_1608Metric, F.Cu at (210.0, 172.1)
- added C66: 1n, Capacitor_SMD:C_0603_1608Metric, F.Cu at (210.0, 174.6)
- added C67: 1u, Capacitor_SMD:C_0603_1608Metric, F.Cu at (216.0, 154.5)
- added C68: 100n, Capacitor_SMD:C_0603_1608Metric, F.Cu at (216.0, 157.0)
- added C69: 1n, Capacitor_SMD:C_0603_1608Metric, F.Cu at (216.0, 159.5)
- added FB5: Bead, Inductor_SMD:L_0603_1608Metric, F.Cu at (216.0, 162.0)
- added J4: Conn_Coaxial, Connector_Coaxial:SMA_Samtec_SMA-J-P-X-ST-EM1_EdgeMount, F.Cu at (224.6, 156.6)
- added L10: 22n, Inductor_SMD:L_0603_1608Metric, F.Cu at (224.0, 181.6)
- added L6: 27n, Inductor_SMD:L_0603_1608Metric, F.Cu at (220.0, 181.6)
- added L7: 56n, Inductor_SMD:L_0603_1608Metric, F.Cu at (224.0, 174.1)
- added L8: 27n, Inductor_SMD:L_0603_1608Metric, F.Cu at (224.0, 176.6)
- added L9: 15n, Inductor_SMD:L_0603_1608Metric, F.Cu at (224.0, 179.1)
- added R34: ~, Parts:HALF_FLANGE_DUMMY_LOAD, F.Cu at (198.1, 173.3)
- added R35: 10k, Resistor_SMD:R_0603_1608Metric, F.Cu at (216.0, 164.6)
- added R36: 10k, Resistor_SMD:R_0603_1608Metric, F.Cu at (216.0, 167.1)
- added R37: 10k, Resistor_SMD:R_0603_1608Metric, F.Cu at (216.0, 169.6)
- C39, C48: value 1u -> 47n
- C40, C42, C45: value 100n -> 47n
- C41, C44, C46, C47: value 1n -> 47n
- C43: value 1n -> 1n5
- C49: value 100n -> 5p1
- C50: value 1n -> 100n
- R26, R28: value 52R3 -> 100R
- R27: value 499R -> 100R
- R29: value 499R -> 56k
- R30: value ~ -> 52R3; footprint Parts:HALF_FLANGE_DUMMY_LOAD -> Resistor_SMD:R_0603_1608Metric
- R31, R33: value 10k -> 499R
- R32: value 10k -> 52R3
- moved J2 211.0 mm to (315.4, 94.0), turned to 90 degrees
- moved J3 41.4 mm to (104.1, 123.2)
Connections:
- net /RF PA/PWR_SP renamed /MCU/RF_PWR_SP
- C39 pad 1: /Exciter/3.3V_IN -> /Receiver/RX_3V3
- C40 pad 1: Net-(U11-CLPF) -> /Receiver/RX_3V3
- C41 pad 1: GND -> /Receiver/RX_3V3
- C41 pad 2: Net-(U11-INLO) -> GND
- C42 pad 1: /RF detectors/RF_DET_3V3 -> /Receiver/RX_3V3
- C43 pad 1: /RF coupler/FWD_SENSE -> Net-(U10-LPF0)
- C43 pad 2: Net-(U11-INHI) -> Net-(U10-LPF1)
- C44 pad 1: /RF detectors/RF_DET_3V3 -> /Receiver/RX_3V3
- C45 pad 1: Net-(U12-CLPF) -> /Receiver/RX_3V3
- C46 pad 1: GND -> /Receiver/RX_3V3
- C46 pad 2: Net-(U12-INLO) -> GND
- C47 pad 1: /RF coupler/REF_SENSE -> /Receiver/RX_3V3
- C47 pad 2: Net-(U12-INHI) -> GND
- C48 pad 1: /Exciter/3.3V_IN -> /Receiver/RX_3V3
- C49 pad 1: /Interface/INTERFACE_3V3 -> Net-(U10-LNA_P)
- C49 pad 2: GND -> Net-(C49-Pad2)
- C50 pad 1: /Interface/INTERFACE_3V3 -> /Exciter/3.3V_IN
- FB3 pad 1: /Exciter/3.3V_IN -> /Receiver/RX_3V3
- FB3 pad 2: /RF detectors/RF_DET_3V3 -> /Exciter/3.3V_IN
- FB4 pad 2: /Interface/INTERFACE_3V3 -> /RF detectors/RF_DET_3V3
- J3 pad 12: /Interface/PA_ENA -> /Interface/PA_EN
- R15 pad 1: /RF PA/PA_EN -> /Interface/PA_EN
- R21 pad 2: /Exciter/SPI_SCK -> /SPI_SCK
- R22 pad 2: /Exciter/SPI_MOSI -> /SPI_MOSI
- R23 pad 2: /Exciter/SPI_MISO -> /SPI_MISO
- R26 pad 1: GND -> Net-(U10-SCLK)
- R26 pad 2: /RF coupler/FWD_SENSE -> /SPI_SCK
- R27 pad 1: Net-(U11-TADJ) -> Net-(U10-SI)
- R27 pad 2: GND -> /SPI_MOSI
- R28 pad 1: GND -> Net-(U10-SO(GPIO1))
- R28 pad 2: /RF coupler/REF_SENSE -> /SPI_MISO
- R29 pad 1: Net-(U12-TADJ) -> Net-(U10-RBIAS)
- R30 pad 1: Net-(R30-In) -> GND
- R31 pad 1: /nRST -> Net-(U11-TADJ)
- R32 pad 1: /TX_nCS -> GND
- R32 pad 2: /Interface/INTERFACE_3V3 -> /RF coupler/REF_SENSE
- R33 pad 1: /RX_nCS -> Net-(U12-TADJ)
- R33 pad 2: /Interface/INTERFACE_3V3 -> GND
- U10 pad 1: unconnected-(U10-VDD_GUARD-Pad1) -> /Receiver/RX_3V3
- U10 pad 11: unconnected-(U10-~{CS}-Pad11) -> /RX_nCS
- U10 pad 12: unconnected-(U10-DVDD-Pad12) -> /Receiver/RX_3V3
- U10 pad 13: unconnected-(U10-AVDD_IF-Pad13) -> /Receiver/RX_3V3
- U10 pad 14: unconnected-(U10-RBIAS-Pad14) -> Net-(U10-RBIAS)
- U10 pad 15: unconnected-(U10-AVDD_RF-Pad15) -> /Receiver/RX_3V3
- U10 pad 17: unconnected-(U10-PA-Pad17) -> /Receiver/RX_3V3
- U10 pad 19: unconnected-(U10-LNA_P-Pad19) -> Net-(U10-LNA_P)
- U10 pad 2: unconnected-(U10-~{RESET}-Pad2) -> /nRST
- U10 pad 20: unconnected-(U10-LNA_N-Pad20) -> Net-(U10-LNA_N)
- U10 pad 21: unconnected-(U10-DCPL_VCO-Pad21) -> Net-(U10-DCPL_VCO)
- U10 pad 22: unconnected-(U10-AVDD_SYNTH1-Pad22) -> /Receiver/RX_3V3
- U10 pad 23: unconnected-(U10-LPF0-Pad23) -> Net-(U10-LPF0)
- U10 pad 24: unconnected-(U10-LPF1-Pad24) -> Net-(U10-LPF1)
- U10 pad 25: unconnected-(U10-AVDD_PFD_CHP-Pad25) -> /Receiver/RX_3V3
- U10 pad 26: unconnected-(U10-DCPL_PFD_CHP-Pad26) -> Net-(U10-DCPL_PFD_CHP)
- U10 pad 27: unconnected-(U10-AVDD_SYNTH2-Pad27) -> /Receiver/RX_3V3
- U10 pad 28: unconnected-(U10-AVDD_XOSC-Pad28) -> /Receiver/RX_3V3
- U10 pad 29: unconnected-(U10-DCPL_XOSC-Pad29) -> Net-(U10-DCPL_XOSC)
- U10 pad 33: unconnected-(U10-GND_EP-Pad33) -> GND
- U10 pad 5: unconnected-(U10-DVDD-Pad5) -> /Receiver/RX_3V3
- U10 pad 6: unconnected-(U10-DCPL-Pad6) -> Net-(U10-DCPL)
- U10 pad 7: unconnected-(U10-SI-Pad7) -> Net-(U10-SI)
- U10 pad 8: unconnected-(U10-SCLK-Pad8) -> Net-(U10-SCLK)
- U10 pad 9: unconnected-(U10-SO(GPIO1)-Pad9) -> Net-(U10-SO(GPIO1))
- U14 pad 3: Net-(R30-In) -> Net-(R34-In)
- U6 pad 11: /Exciter/SPI_nCS -> /TX_nCS
- U6 pad 2: /Exciter/nRST -> /nRST
Other:
- board size 240 x 150 mm -> 255 x 165 mm

Commit message: Add files via upload
Parts:
- added C70: 2u2, Capacitor_SMD:C_0603_1608Metric, F.Cu at (120.8, 68.5)
- added C71: 1u, Capacitor_SMD:C_0603_1608Metric, F.Cu at (120.8, 71.0)
- added C72: 1u, Capacitor_SMD:C_0603_1608Metric, F.Cu at (120.8, 73.5)
- added C73: 100n, Capacitor_SMD:C_0603_1608Metric, F.Cu at (120.8, 76.0)
- added C74: 100n, Capacitor_SMD:C_0603_1608Metric, F.Cu at (124.8, 68.5)
- added C75: 10n, Capacitor_SMD:C_0603_1608Metric, F.Cu at (124.8, 71.0)
- added C76: 10n, Capacitor_SMD:C_0603_1608Metric, F.Cu at (124.8, 73.5)
- added C77: 100n, Capacitor_SMD:C_0603_1608Metric, F.Cu at (124.8, 76.0)
- added C78: 100n, Capacitor_SMD:C_0603_1608Metric, F.Cu at (128.8, 68.5)
- added C79: 100n, Capacitor_SMD:C_0603_1608Metric, F.Cu at (128.8, 71.0)
- added C80: 100n, Capacitor_SMD:C_0603_1608Metric, F.Cu at (128.8, 73.5)
- added C81: 1u, Capacitor_SMD:C_0603_1608Metric, F.Cu at (103.5, 68.5)
- added C82: 100n, Capacitor_SMD:C_0603_1608Metric, F.Cu at (103.5, 71.0)
- added C83: 1n, Capacitor_SMD:C_0603_1608Metric, F.Cu at (103.5, 73.5)
- added FB6: Bead, Inductor_SMD:L_0603_1608Metric, F.Cu at (128.8, 76.0)
- added FB7: Bead, Inductor_SMD:L_0603_1608Metric, F.Cu at (103.5, 76.0)
- added J5: Conn_Coaxial, Connector_Coaxial:SMA_Samtec_SMA-J-P-X-ST-EM1_EdgeMount, F.Cu at (112.1, 70.5)
- added R38: 10k, Resistor_SMD:R_0603_1608Metric, F.Cu at (103.5, 78.5)
- added R39: 10k, Resistor_SMD:R_0603_1608Metric, F.Cu at (103.5, 81.0)
- added R40: 10k, Resistor_SMD:R_0603_1608Metric, F.Cu at (103.5, 83.5)
- added Y1: 12MHz, Crystal:Crystal_SMD_3225-4Pin_3.2x2.5mm, F.Cu at (121.4, 79.5)
- C67: value 1u -> 10p
- C68: value 100n -> 10p
- C69: value 1n -> 2u2
- J3: value Conn_01x16 -> Conn_01x05; footprint Connector_PinHeader_2.54mm:PinHeader_2x08_P2.54mm_Vertical_SMD -> Connector_PinHeader_2.54mm:PinHeader_1x05_P2.54mm_Vertical_SMD_Pin1Left
- J4: value Conn_Coaxial -> Conn_01x16; footprint Connector_Coaxial:SMA_Samtec_SMA-J-P-X-ST-EM1_EdgeMount -> Connector_PinHeader_2.54mm:PinHeader_2x08_P2.54mm_Vertical_SMD
- R34: value ~ -> 100R; footprint Parts:HALF_FLANGE_DUMMY_LOAD -> Resistor_SMD:R_0603_1608Metric
- R35, R36: value 10k -> 100R
- R37: value 10k -> ~; footprint Resistor_SMD:R_0603_1608Metric -> Parts:HALF_FLANGE_DUMMY_LOAD
Connections:
- net /RF coupler/FWD_SENSE renamed /RF coupler/FWD_RF
- net /RF coupler/REF_SENSE renamed /RF coupler/REF_RF
- C67 pad 1: /Exciter/3.3V_IN -> /MCU/OSC1
- C68 pad 1: /Interface/INTERFACE_3V3 -> /MCU/OSC2
- C69 pad 1: /Interface/INTERFACE_3V3 -> Net-(U13-VCAP_1)
- FB5 pad 2: /Interface/INTERFACE_3V3 -> /MCU/MCU_3V3
- J3 pad 1: /nRST -> GND
- J3 pad 2: /SPI_MISO -> /nRST
- J3 pad 3: /SPI_MOSI -> /MCU/SWDIO
- J3 pad 4: /SPI_SCK -> /MCU/SWDCLK
- J3 pad 5: /TX_nCS -> /MCU/MCU_3V3
- J4 pad 1: /RF input filter/RF_OUT -> /nRST
- J4 pad 2: GND -> /SPI_MISO
- R3 pad 1: /RF PA/FWD_SENSE_IN -> /FWD_SENSE
- R34 pad 1: Net-(R34-In) -> Net-(U13-PB3)
- R35 pad 1: /nRST -> Net-(U13-PB4)
- R35 pad 2: GND -> /SPI_MISO
- R36 pad 1: /TX_nCS -> Net-(U13-PB5)
- R36 pad 2: /Interface/INTERFACE_3V3 -> /SPI_MOSI
- R37 pad 1: /RX_nCS -> Net-(R37-In)
- U11 pad 6: /RF PA/FWD_SENSE_IN -> /FWD_SENSE
- U11 pad 7: /RF PA/FWD_SENSE_IN -> /FWD_SENSE
- U12 pad 6: /RF detectors/RF_REF_DET -> /REF_SENSE
- U12 pad 7: /RF detectors/RF_REF_DET -> /REF_SENSE
- U13 pad 1: unconnected-(U13-VBAT-Pad1) -> /MCU/MCU_3V3
- U13 pad 12: unconnected-(U13-VSSA-Pad12) -> GND
- U13 pad 13: unconnected-(U13-VDDA-Pad13) -> /MCU/MCU_VDDA_3V3
- U13 pad 14: unconnected-(U13-PA0-Pad14) -> /FWD_SENSE
- U13 pad 15: unconnected-(U13-PA1-Pad15) -> /REF_SENSE
- U13 pad 16: unconnected-(U13-PA2-Pad16) -> /MCU/AIN2
- U13 pad 17: unconnected-(U13-PA3-Pad17) -> /MCU/AIN3
- U13 pad 18: Net-(U13-VSS-Pad18) -> GND
- U13 pad 19: unconnected-(U13-VDD-Pad19) -> /MCU/MCU_3V3
- U13 pad 20: unconnected-(U13-PA4-Pad20) -> /MCU/RF_PWR_SP
- U13 pad 21: unconnected-(U13-PA5-Pad21) -> /MCU/AOUT1
- U13 pad 31: unconnected-(U13-VCAP_1-Pad31) -> Net-(U13-VCAP_1)
- U13 pad 32: unconnected-(U13-VDD-Pad32) -> /MCU/MCU_3V3
- U13 pad 42: unconnected-(U13-PA9-Pad42) -> /Interface/MCU_TX
- U13 pad 43: unconnected-(U13-PA10-Pad43) -> /Interface/MCU_RX
- U13 pad 46: unconnected-(U13-PA13-Pad46) -> /MCU/SWDIO
- U13 pad 47: unconnected-(U13-VCAP_2-Pad47) -> Net-(U13-VCAP_2)
- U13 pad 48: unconnected-(U13-VDD-Pad48) -> /MCU/MCU_3V3
- U13 pad 49: unconnected-(U13-PA14-Pad49) -> /MCU/SWDCLK
- U13 pad 5: unconnected-(U13-PH0-Pad5) -> /MCU/OSC1
- U13 pad 55: unconnected-(U13-PB3-Pad55) -> Net-(U13-PB3)
- U13 pad 56: unconnected-(U13-PB4-Pad56) -> Net-(U13-PB4)
- U13 pad 57: unconnected-(U13-PB5-Pad57) -> Net-(U13-PB5)
- U13 pad 58: unconnected-(U13-PB6-Pad58) -> /RX_nCS
- U13 pad 59: unconnected-(U13-PB7-Pad59) -> /TX_nCS
- U13 pad 6: unconnected-(U13-PH1-Pad6) -> /MCU/OSC2
- U13 pad 60: unconnected-(U13-BOOT0-Pad60) -> GND
- U13 pad 61: unconnected-(U13-PB8-Pad61) -> /MCU/PA_EN
- U13 pad 63: Net-(U13-VSS-Pad18) -> GND
- U13 pad 64: unconnected-(U13-VDD-Pad64) -> /MCU/MCU_3V3
- U13 pad 7: unconnected-(U13-NRST-Pad7) -> /nRST
- U14 pad 3: Net-(R34-In) -> Net-(R37-In)

Commit message: Add files via upload
Parts:
- added J6: Conn_Coaxial, Connector_Coaxial:SMA_Samtec_SMA-J-P-X-ST-EM1_EdgeMount, F.Cu at (318.2, 143.0)
- added JP1: ~, Jumper:SolderJumper-2_P1.3mm_Open_TrianglePad1.0x1.5mm, F.Cu at (182.1, 194.0)
- added Q3: NP100P04PDG, Package_TO_SOT_SMD:TO-263-2, F.Cu at (184.6, 184.1)
- added R41: 10k, Resistor_SMD:R_0603_1608Metric, F.Cu at (175.9, 193.5)
- added R42: 10k, Resistor_SMD:R_0603_1608Metric, F.Cu at (175.9, 196.0)
- added R43: 10k, Resistor_SMD:R_0603_1608Metric, F.Cu at (175.9, 198.5)
- added TP9: ~, TestPoint:TestPoint_Pad_D1.5mm, F.Cu at (188.0, 194.0)
- J4: value Conn_01x16 -> Conn_01x05; footprint Connector_PinHeader_2.54mm:PinHeader_2x08_P2.54mm_Vertical_SMD -> Connector_PinHeader_2.54mm:PinHeader_1x05_P2.54mm_Vertical_SMD_Pin1Left
- J5: value Conn_Coaxial -> Conn_01x16; footprint Connector_Coaxial:SMA_Samtec_SMA-J-P-X-ST-EM1_EdgeMount -> Connector_PinHeader_2.54mm:PinHeader_2x08_P2.54mm_Vertical_SMD
- Q2: value NP100P04PDG -> BSS138; footprint Package_TO_SOT_SMD:TO-263-2 -> Package_TO_SOT_SMD:SOT-23
- R16, R38, R39: value 10k -> 100R
- R17: value 47k -> 10k
- R19: value 24k -> 10k
- R20: value 75k -> 12k
- R21: value 100R -> 100k
- R22: value 100R -> 24k
- R23: value 100R -> 75k
- R24, R29: value 56k -> 100R
- R25: value 18R -> 100R
- R27: value 100R -> 56k
- R28: value 100R -> 18R
- R30: value 52R3 -> 100R
- R31: value 499R -> 100R
- R32: value 52R3 -> 56k
- R33: value 499R -> 52R3
- R34, R36: value 100R -> 499R
- R35: value 100R -> 52R3
- R37: value ~ -> 100R; footprint Parts:HALF_FLANGE_DUMMY_LOAD -> Resistor_SMD:R_0603_1608Metric
- R40: value 10k -> ~; footprint Resistor_SMD:R_0603_1608Metric -> Parts:HALF_FLANGE_DUMMY_LOAD
- moved R40 168.0 mm to (264.0, 133.0)
- moved R37 46.6 mm to (215.8, 123.0)
- moved U13 12.9 mm to (238.0, 130.0)
Connections:
- J3 pad 1: GND -> /MCU/TP1
- J3 pad 2: /nRST -> /MCU/TP2
- J3 pad 3: /MCU/SWDIO -> /MCU/DBG_TX
- J3 pad 4: /MCU/SWDCLK -> /MCU/DBG_RX
- J3 pad 5: /MCU/MCU_3V3 -> GND
- J4 pad 1: /nRST -> GND
- J4 pad 2: /SPI_MISO -> /nRST
- J4 pad 3: /SPI_MOSI -> /MCU/SWDIO
- J4 pad 4: /SPI_SCK -> /MCU/SWDCLK
- J4 pad 5: /TX_nCS -> /MCU/MCU_3V3
- J5 pad 1: /RF input filter/RF_OUT -> /nRST
- J5 pad 2: GND -> /SPI_MISO
- Q1 pad 2: GND -> Net-(Q1-S)
- Q2 pad 1: Net-(Q1-D) -> Net-(Q2-G)
- Q2 pad 2: /RF PA/RF_PA_VDD -> GND
- Q2 pad 3: /Power supply/13.8V_OUT -> Net-(Q1-S)
- R16 pad 1: GND -> /MCU/PA_EN
- R16 pad 2: Net-(Q1-G) -> Net-(Q2-G)
- R17 pad 1: Net-(Q1-D) -> Net-(Q1-S)
- R17 pad 2: /Power supply/13.8V_OUT -> Net-(Q1-G)
- R18 pad 1: /Power supply/13.8V_OUT -> Net-(Q2-G)
- R18 pad 2: Net-(U5-EN) -> Net-(Q1-S)
- R19 pad 1: Net-(U5-FB) -> GND
- R19 pad 2: GND -> Net-(Q2-G)
- R20 pad 1: Net-(U5-FB) -> Net-(Q1-D)
- R20 pad 2: /Exciter/3.3V_IN -> /Power supply/13.8V_OUT
- R21 pad 1: Net-(U6-SCLK) -> /Power supply/13.8V_OUT
- R21 pad 2: /SPI_SCK -> Net-(U5-EN)
- R22 pad 1: Net-(U6-SI) -> Net-(U5-FB)
- R22 pad 2: /SPI_MOSI -> GND
- R23 pad 1: Net-(U6-SO(GPIO1)) -> Net-(U5-FB)
- R23 pad 2: /SPI_MISO -> /Exciter/3.3V_IN
- R24 pad 1: Net-(U6-RBIAS) -> Net-(U6-SCLK)
- R24 pad 2: GND -> /SPI_SCK
- R25 pad 1: Net-(C33-Pad2) -> Net-(U6-SI)
- R25 pad 2: /Exciter/EXCITER_3V3 -> /SPI_MOSI
- R26 pad 1: Net-(U10-SCLK) -> Net-(U6-SO(GPIO1))
- R26 pad 2: /SPI_SCK -> /SPI_MISO
- R27 pad 1: Net-(U10-SI) -> Net-(U6-RBIAS)
- R27 pad 2: /SPI_MOSI -> GND
- R28 pad 1: Net-(U10-SO(GPIO1)) -> Net-(C33-Pad2)
- R28 pad 2: /SPI_MISO -> /Exciter/EXCITER_3V3
- R29 pad 1: Net-(U10-RBIAS) -> Net-(U10-SCLK)
- R29 pad 2: GND -> /SPI_SCK
- R30 pad 1: GND -> Net-(U10-SI)
- R30 pad 2: /RF coupler/FWD_RF -> /SPI_MOSI
- R31 pad 1: Net-(U11-TADJ) -> Net-(U10-SO(GPIO1))
- R31 pad 2: GND -> /SPI_MISO
- R32 pad 1: GND -> Net-(U10-RBIAS)
- R32 pad 2: /RF coupler/REF_RF -> GND
- R33 pad 1: Net-(U12-TADJ) -> GND
- R33 pad 2: GND -> /RF coupler/FWD_RF
- R34 pad 1: Net-(U13-PB3) -> Net-(U11-TADJ)
- R34 pad 2: /SPI_SCK -> GND
- R35 pad 1: Net-(U13-PB4) -> GND
- R35 pad 2: /SPI_MISO -> /RF coupler/REF_RF
- R36 pad 1: Net-(U13-PB5) -> Net-(U12-TADJ)
- R36 pad 2: /SPI_MOSI -> GND
- R37 pad 1: Net-(R37-In) -> Net-(U13-PB3)
- R38 pad 1: /nRST -> Net-(U13-PB4)
- R38 pad 2: GND -> /SPI_MISO
- R39 pad 1: /TX_nCS -> Net-(U13-PB5)
- R39 pad 2: /Interface/INTERFACE_3V3 -> /SPI_MOSI
- R40 pad 1: /RX_nCS -> Net-(R40-In)
- TP6 pad 1: Net-(Q1-D) -> Net-(Q2-G)
- TP7 pad 1: /Power supply/13.8V_OUT -> Net-(Q1-D)
- TP8 pad 1: /Exciter/3.3V_IN -> /Power supply/13.8V_OUT
- U10 pad 17: /Receiver/RX_3V3 -> Net-(JP1-B)
- U13 pad 27: unconnected-(U13-PB1-Pad27) -> /MCU/TP1
- U13 pad 28: unconnected-(U13-PB2-Pad28) -> /MCU/TP2
- U13 pad 29: unconnected-(U13-PB10-Pad29) -> /MCU/DBG_TX
- U13 pad 30: unconnected-(U13-PB11-Pad30) -> /MCU/DBG_RX
- U14 pad 3: Net-(R37-In) -> Net-(R40-In)
