File: rf_in_flt.kicad_sch (KiCad schematic)
At the start: 1 part, among them J2 N_PAD

Commit message: date update
Other:
- title: M17 Remote Radio Unit - RF board -> Remote Radio Unit - RF board
Changed lines of the file:
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@@
   (paper "A3")
   (title_block
-    (title "M17 Remote Radio Unit - RF board")
-    (date "28-10-2023")
+    (title "Remote Radio Unit - RF board")
+    (date "30-10-2023")
     (rev "A")
     (company "M17 Project")

Commit message: MPN/PN update
Parts:
- J2: MPN (none) -> -
Changed lines of the file:
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@@
+      (effects (font (size 1.27 1.27)) hide)
+    )
+    (property "MPN" "-" (at 215.9 138.43 0)
       (effects (font (size 1.27 1.27)) hide)
     )
