File: circ.kicad_sch (KiCad schematic)
At the start: 2 parts, among them U16 WH3538X-1

Commit message: WIP rev C
Parts:
- renumbered U16 to U15
Changed lines of the file:
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@@
   (title_block
     (title "Remote Radio Unit - RF board")
-    (date "20-01-2024")
-    (rev "B")
+    (date "04-04-2024")
+    (rev "C")
     (company "M17 Project")
     (comment 1 "Wojciech Kaczmarski, SP5WWP")
@@
   (symbol (lib_id "Parts:WH3538X-1") (at 203.2 127 0) (unit 1)
     (in_bom yes) (on_board yes) (dnp no) (fields_autoplaced)
-    (property "Reference" "U16" (at 203.0795 115.4879 0)
+    (property "Reference" "U15" (at 203.0795 115.4879 0)
       (effects (font (size 1.27 1.27)))
     )
@@
       (project "m17-rru-rf"
         (path "/4c42207c-9e6b-42da-ad38-da126b892014/52ad0992-68c2-4318-a1ac-e7f0506bc4fb"
-          (reference "U16") (unit 1)
+          (reference "U15") (unit 1)
         )
       )
