File: rf_cpl.kicad_sch (KiCad schematic)
At the start: 4 parts, among them J3 N_PAD, U10 SYBD-30-62HP+, U11 GAT-30+, U9 GAT-30+

Commit message: WIP rev C
Parts:
- renumbered U11 to U10, U9 to U8, U10 to U9
Changed lines of the file:
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@@
   (title_block
     (title "Remote Radio Unit - RF board")
-    (date "20-01-2024")
-    (rev "B")
+    (date "04-04-2024")
+    (rev "C")
     (company "M17 Project")
     (comment 1 "Wojciech Kaczmarski, SP5WWP")
@@
   (symbol (lib_id "power:GND") (at 182.88 154.94 0) (unit 1)
     (in_bom yes) (on_board yes) (dnp no) (fields_autoplaced)
-    (property "Reference" "#PWR065" (at 182.88 161.29 0)
+    (property "Reference" "#PWR071" (at 182.88 161.29 0)
       (effects (font (size 1.27 1.27)) hide)
     )
@@
       (project "m17-rru-rf"
         (path "/4c42207c-9e6b-42da-ad38-da126b892014/59b2721c-5b8a-4fc3-bf5e-590dec787afb"
-          (reference "#PWR065") (unit 1)
+          (reference "#PWR071") (unit 1)
         )
       )
@@
   (symbol (lib_id "power:GND") (at 242.57 135.89 0) (unit 1)
     (in_bom yes) (on_board yes) (dnp no) (fields_autoplaced)
-    (property "Reference" "#PWR068" (at 242.57 142.24 0)
+    (property "Reference" "#PWR074" (at 242.57 142.24 0)
       (effects (font (size 1.27 1.27)) hide)
     )
@@
       (project "m17-rru-rf"
         (path "/4c42207c-9e6b-42da-ad38-da126b892014/59b2721c-5b8a-4fc3-bf5e-590dec787afb"
-          (reference "#PWR068") (unit 1)
+          (reference "#PWR074") (unit 1)
         )
       )
@@
   (symbol (lib_id "Parts:GAT-30+") (at 223.52 151.13 270) (unit 1)
     (in_bom yes) (on_board yes) (dnp no) (fields_autoplaced)
-    (property "Reference" "U11" (at 229.235 151.13 90)
+    (property "Reference" "U10" (at 229.235 151.13 90)
       (effects (font (size 1.27 1.27)) (justify left))
     )
@@
       (project "m17-rru-rf"
         (path "/4c42207c-9e6b-42da-ad38-da126b892014/59b2721c-5b8a-4fc3-bf5e-590dec787afb"
-          (reference "U11") (unit 1)
+          (reference "U10") (unit 1)
         )
       )
@@
   (symbol (lib_id "Parts:GAT-30+") (at 193.04 151.13 270) (unit 1)
     (in_bom yes) (on_board yes) (dnp no) (fields_autoplaced)
-    (property "Reference" "U9" (at 198.755 151.13 90)
+    (property "Reference" "U8" (at 198.755 151.13 90)
       (effects (font (size 1.27 1.27)) (justify left))
     )
@@
       (project "m17-rru-rf"
         (path "/4c42207c-9e6b-42da-ad38-da126b892014/59b2721c-5b8a-4fc3-bf5e-590dec787afb"
-          (reference "U9") (unit 1)
+          (reference "U8") (unit 1)
         )
       )
@@
   (symbol (lib_id "Parts:SYBD-30-62HP+") (at 208.28 127 0) (mirror y) (unit 1)
     (in_bom yes) (on_board yes) (dnp no)
-    (property "Reference" "U10" (at 208.28 123.19 0)
+    (property "Reference" "U9" (at 208.28 123.19 0)
       (effects (font (size 1.27 1.27)))
     )
@@
       (project "m17-rru-rf"
         (path "/4c42207c-9e6b-42da-ad38-da126b892014/59b2721c-5b8a-4fc3-bf5e-590dec787afb"
-          (reference "U10") (unit 1)
+          (reference "U9") (unit 1)
         )
       )
@@
   (symbol (lib_id "power:GND") (at 208.28 138.43 0) (unit 1)
     (in_bom yes) (on_board yes) (dnp no) (fields_autoplaced)
-    (property "Reference" "#PWR066" (at 208.28 144.78 0)
+    (property "Reference" "#PWR072" (at 208.28 144.78 0)
       (effects (font (size 1.27 1.27)) hide)
     )
@@
       (project "m17-rru-rf"
         (path "/4c42207c-9e6b-42da-ad38-da126b892014/59b2721c-5b8a-4fc3-bf5e-590dec787afb"
-          (reference "#PWR066") (unit 1)
+          (reference "#PWR072") (unit 1)
         )
       )
@@
   (symbol (lib_id "power:GND") (at 213.36 154.94 0) (unit 1)
     (in_bom yes) (on_board yes) (dnp no) (fields_autoplaced)
-    (property "Reference" "#PWR067" (at 213.36 161.29 0)
+    (property "Reference" "#PWR073" (at 213.36 161.29 0)
       (effects (font (size 1.27 1.27)) hide)
     )
@@
       (project "m17-rru-rf"
         (path "/4c42207c-9e6b-42da-ad38-da126b892014/59b2721c-5b8a-4fc3-bf5e-590dec787afb"
-          (reference "#PWR067") (unit 1)
-        )
-      )
+          (reference "#PWR073") (unit 1)
+        )
+      )

Commit message: KiCAD version bump to 8.0.2
- updated U9 PN
Parts:
- U9: MPN - -> SYBD-30-62HP+; PN - -> SYBD-30-62HP+
